File: KiCad/ATI DNA-C PCB Smart PWM v3/ATI DNA-C PCB Smart PWM v3.kicad_pcb (KiCad board)
At the start: 2 copper layers, 70 x 20 mm, 18 parts, among them U1 SmartPWMv3

Commit message: More Derp - Fixed
Other:
- board text removed: "Designed by MosMax"
- board text removed: "Powered by"
Changed lines of the file:
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@@
   (general
     (thickness 1.6)
-    (drawings 37)
+    (drawings 32)
     (tracks 81)
     (zones 0)
@@
     )
   )
-  (gr_text "Designed by MosMax" (at 161.69 95.29) (layer B.SilkS)
-    (effects (font (size 1 1) (thickness 0.15)) (justify mirror))
-  )
-  (gr_text "Powered by" (at 163.95 97.99) (layer B.SilkS)
-    (effects (font (size 1 1) (thickness 0.15)) (justify mirror))
-  )
-  (gr_poly (pts (xy 156.694106 97.747276) (xy 156.913181 97.743307) (xy 156.360731 96.847163) (xy 156.357556 96.843988) (xy 156.235319 96.647138) (xy 156.210712 96.647138) (xy 155.713031 96.647138) (xy 155.683662 96.647138) (xy 155.458237 96.647138) (xy 155.601113 96.853513) (xy 155.6027 96.853513) (xy 155.867812 97.2742) (xy 155.871781 97.278169) (xy 155.990843 97.469463) (xy 156.043231 97.469463) (xy 156.417087 97.47105) (xy 156.278181 97.282138) (xy 156.101968 97.282138) (xy 156.101175 97.278963) (xy 156.098 97.274994) (xy 155.83765 96.853513) (xy 156.128162 96.853513) (xy 156.694106 97.747276)) (layer B.SilkS) (width 0.007937))
-  (gr_poly (pts (xy 157.214806 98.250513) (xy 156.966363 98.250513) (xy 157.358475 98.952188) (xy 158.558625 96.889232) (xy 158.844375 96.894788) (xy 158.6634 97.218638) (xy 158.459406 97.218638) (xy 158.3205 97.472638) (xy 158.765 97.472638) (xy 159.245219 96.647138) (xy 158.425275 96.647138) (xy 157.352918 98.495782) (xy 157.214806 98.250513)) (layer B.SilkS) (width 0.007937))
-  (gr_poly (pts (xy 157.610887 97.869513) (xy 156.163087 97.869513) (xy 157.364824 99.924532) (xy 158.540368 97.869513) (xy 158.063325 97.869513) (xy 157.931562 98.107638) (xy 158.142699 98.107638) (xy 157.356887 99.410181) (xy 156.595681 98.123513) (xy 157.452931 98.123513) (xy 157.610887 97.869513)) (layer B.SilkS) (width 0.007937))
   (dimension 65.99954 (width 0.12) (layer F.Fab)
     (gr_text "66.000 mm" (at 151.527722 132.664093 -0.2) (layer F.Fab)
