File: KiCad/VoltMax PWM/VoltMax PWM.sch (KiCad schematic (older format))
At the start: 28 parts, among them IC1 DS1809Z-010+, IC2 NCV4264-2ST50T3G, J1 BAT-, J2 510-, J3 VIN+, J4 PAD_Fire2, J5 PAD_Fire1, J6 VM-, J7 VM+, Q1 SSM3J334R_LF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

Commit message: Better thermal, cleaner vias/traces
Connections:
- net labels added: S4VIN+toS1
- net labels removed: VIN+toFire1
- wire segments 102 -> 108
Other:
- moved on the sheet: D3, R5
Changed lines of the file:
@@
 Wire Wire Line
 	6350 4200 6950 4200
-Text Label 5100 4800 1    50   ~ 0
+Text Label 4950 4800 1    50   ~ 0
 VIN+toQ1Drain
 Connection ~ 6950 5050
@@
 L Device:R R5
 U 1 1 5CAAB1BD
-P 5450 3850
-F 0 "R5" V 5657 3850 50  0000 C CNN
-F 1 "570" V 5566 3850 50  0000 C CNN
-F 2 "VoltMax PWM:R_0603_1608Metric" V 5380 3850 50  0001 C CNN
-F 3 "~" H 5450 3850 50  0001 C CNN
-	1    5450 3850
+P 5550 3850
+F 0 "R5" V 5757 3850 50  0000 C CNN
+F 1 "570" V 5666 3850 50  0000 C CNN
+F 2 "VoltMax PWM:R_0603_1608Metric" V 5480 3850 50  0001 C CNN
+F 3 "~" H 5550 3850 50  0001 C CNN
+	1    5550 3850
 	0    1    1    0
 $EndComp
@@
 L Device:LED D3
 U 1 1 5CAACF2D
-P 5850 3850
-F 0 "D3" H 5850 4050 50  0000 C CNN
-F 1 "LED" H 5850 3950 50  0000 C CNN
-F 2 "VoltMax PWM:LED_4mm" H 5850 3850 50  0001 C CNN
-F 3 "~" H 5850 3850 50  0001 C CNN
-	1    5850 3850
+P 5950 3850
+F 0 "D3" H 5950 4050 50  0000 C CNN
+F 1 "LED" H 5950 3950 50  0000 C CNN
+F 2 "VoltMax PWM:LED_4mm" H 5950 3850 50  0001 C CNN
+F 3 "~" H 5950 3850 50  0001 C CNN
+	1    5950 3850
 	-1   0    0    1
 $EndComp
 Wire Wire Line
-	5400 3500 5300 3500
-Wire Wire Line
-	5300 3500 5300 3850
-Wire Wire Line
-	5600 3850 5700 3850
-Wire Wire Line
-	6500 3850 6500 4800
-Wire Wire Line
-	6000 3850 6500 3850
+	5700 3850 5800 3850
 $Comp
 L VoltMax~PWM:SS12D07VG4NSGAPA S4
@@
 Text Label 5500 3050 0    50   ~ 0
 VIN+toSwitch
-Text Label 6250 3850 0    50   ~ 0
-VIN+toFire1
-Text Label 5650 3850 3    50   ~ 0
+Text Label 5750 3850 3    50   ~ 0
 R5toD3
 Text Label 4500 5150 0    50   ~ 0
 GatetoGND
-Text Label 5300 3500 3    50   ~ 0
+Text Label 5300 3800 3    50   ~ 0
 VIN+toR5
 Text Label 4000 3900 1    50   ~ 0
@@
 Wire Wire Line
 	1650 2700 2050 2700
+Connection ~ 7000 2000
+$Comp
+L power:GND #PWR0102
+U 1 1 5CB29115
+P 6650 3400
+F 0 "#PWR0102" H 6650 3150 50  0001 C CNN
+F 1 "GND" H 6655 3227 50  0000 C CNN
+F 2 "" H 6650 3400 50  0001 C CNN
+F 3 "" H 6650 3400 50  0001 C CNN
+	1    6650 3400
+	-1   0    0    1
+$EndComp
+Text GLabel 6650 3550 2    50   Input ~ 0
+GND
+Wire Wire Line
+	6650 3400 6650 3850
+Wire Wire Line
+	6100 3850 6650 3850
+Wire Wire Line
+	5150 3500 5150 5200
+Wire Wire Line
+	5150 5200 6650 5200
+Wire Wire Line
+	6650 5200 6650 4800
+Wire Wire Line
+	6650 4800 6500 4800
+Text Label 5400 5200 3    50   ~ 0
+S4VIN+toS1
+Wire Wire Line
+	5400 3850 5300 3850
+Wire Wire Line
+	5150 3500 5300 3500
+Wire Wire Line
+	5300 3850 5300 3500
+Connection ~ 5300 3500
+Wire Wire Line
+	5300 3500 5400 3500
 $EndSCHEMATC

Commit message: David has spoken and changes have been made, cleaner vias/traces
Parts:
- removed R4: 1K, VoltMax PWM:R_0603_1608Metric, symbol Device:R
- R2: value 1M -> 10K
- renumbered R5 to R4
Connections:
- net labels added: CStoR2, S1toVS, U1toS1, VIN+toS4
- net labels removed: R2toVS, S4VIN+toS1, U1toR2, VIN+toQ1Drain
- wire segments 108 -> 114
Other:
- moved on the sheet: J4, J5, R2
Changed lines of the file:
@@
 	4300 4800 4150 4800
-Wire Wire Line
-	2700 4300 2750 4300
 Wire Wire Line
 	2250 4200 2750 4200
@@
 	2750 3900 2250 3900
 Connection ~ 2250 3900
-Wire Wire Line
-	3750 4100 3900 4100
-Wire Wire Line
-	3900 4100 3900 4800
-Connection ~ 3900 4800
-Wire Wire Line
-	2250 5400 2250 4200
-Connection ~ 2250 4200
-Wire Wire Line
-	2700 4300 2700 4800
-Wire Wire Line
-	2700 4800 3100 4800
 Text Label 6950 3050 0    50   ~ 0
 510-
 Wire Wire Line
 	6350 4200 6950 4200
-Text Label 4950 4800 1    50   ~ 0
-VIN+toQ1Drain
+Text Label 5150 4400 2    50   ~ 0
+VIN+toS4
 Connection ~ 6950 5050
 Wire Wire Line
@@
 L power:GND #PWR01
 U 1 1 5C9E7679
-P 2250 5400
-F 0 "#PWR01" H 2250 5150 50  0001 C CNN
-F 1 "GND" H 2255 5227 50  0000 C CNN
-F 2 "" H 2250 5400 50  0001 C CNN
-F 3 "" H 2250 5400 50  0001 C CNN
-	1    2250 5400
+P 1950 4950
+F 0 "#PWR01" H 1950 4700 50  0001 C CNN
+F 1 "GND" H 1955 4777 50  0000 C CNN
+F 2 "" H 1950 4950 50  0001 C CNN
+F 3 "" H 1950 4950 50  0001 C CNN
+	1    1950 4950
 	1    0    0    -1
 $EndComp
@@
 	1    6200 4200
 	0    -1   -1   0
-$EndComp
-$Comp
-L Device:R R2
-U 1 1 5C9B0658
-P 3250 4800
-F 0 "R2" V 3043 4800 50  0000 C CNN
-F 1 "1M" V 3134 4800 50  0000 C CNN
-F 2 "VoltMax PWM:R_0603_1608Metric" V 3180 4800 50  0001 C CNN
-F 3 "~" H 3250 4800 50  0001 C CNN
-	1    3250 4800
-	0    1    1    0
 $EndComp
 $Comp
@@
 L VoltMax~PWM:KSC641JLFS S1
 U 1 1 5C9BEA02
-P 6500 4900
-F 0 "S1" H 7100 5165 50  0000 C CNN
-F 1 "KSC641JLFS" H 7100 5074 50  0000 C CNN
-F 2 "KSC641JLFS" H 7550 5000 50  0001 L CNN
-F 3 "" H 7550 4900 50  0001 L CNN
-F 4 "1 Way Surface Mount DIP & SIP Switch SPST-NO, Plunger Actuator, IP67" H 7550 4800 50  0001 L CNN "Description"
-F 5 "2" H 7550 4700 50  0001 L CNN "Height"
-F 6 "KSC641JLFS" H 7550 4500 50  0001 L CNN "Manufacturer_Part_Number"
-	1    6500 4900
+P 3800 5100
+F 0 "S1" H 4400 5365 50  0000 C CNN
+F 1 "KSC641JLFS" H 4400 5274 50  0000 C CNN
+F 2 "KSC641JLFS" H 4850 5200 50  0001 L CNN
+F 3 "" H 4850 5100 50  0001 L CNN
+F 4 "1 Way Surface Mount DIP & SIP Switch SPST-NO, Plunger Actuator, IP67" H 4850 5000 50  0001 L CNN "Description"
+F 5 "2" H 4850 4900 50  0001 L CNN "Height"
+F 6 "KSC641JLFS" H 4850 4700 50  0001 L CNN "Manufacturer_Part_Number"
+	1    3800 5100
 	-1   0    0    1
 $EndComp
-Wire Wire Line
-	5300 4900 5300 4800
 $Comp
 L VoltMax~PWM:KSC641JLFS S3
@@
 Connection ~ 4950 4200
 Wire Wire Line
-	4950 4200 4950 4100
-$Comp
-L Device:R R4
-U 1 1 5C9B1043
-P 4950 3950
-F 0 "R4" H 5020 3996 50  0000 L CNN
-F 1 "1K" H 5020 3905 50  0000 L CNN
-F 2 "VoltMax PWM:R_0603_1608Metric" V 4880 3950 50  0001 C CNN
-F 3 "~" H 4950 3950 50  0001 C CNN
-	1    4950 3950
-	1    0    0    -1
-$EndComp
-Wire Wire Line
 	4650 1450 4950 1450
 Wire Wire Line
@@
 Down
 Wire Wire Line
-	3400 4800 3900 4800
-Connection ~ 5300 4800
-Wire Wire Line
-	6500 4900 6500 4800
-Connection ~ 6500 4800
-Wire Wire Line
 	800  1350 3650 1350
 Wire Wire Line
@@
 Wire Wire Line
 	3100 2450 4150 2450
-Wire Wire Line
-	4950 1450 4950 3800
 Wire Wire Line
 	2050 2700 2050 2450
@@
 	7000 2000 7000 850
 Wire Wire Line
-	4650 850  7000 850
+	4650 850  5050 850
 Wire Wire Line
 	7000 2000 7150 2000
@@
 Connection ~ 5400 2300
 Wire Wire Line
-	4900 4800 5300 4800
-Wire Wire Line
-	4000 4800 4000 3050
-Wire Wire Line
 	4000 3050 5150 3050
-Connection ~ 4000 4800
-Wire Wire Line
-	4000 4800 3900 4800
 $Comp
 L Connector_Generic:Conn_01x01 J1
@@
 Text GLabel 4500 5250 0    50   Input ~ 0
 GND
-Text GLabel 2250 5250 0    50   Input ~ 0
+Text GLabel 1950 4800 0    50   Input ~ 0
 GND
 Text GLabel 4150 2550 0    50   Input ~ 0
@@
 L Connector_Generic:Conn_01x01 J5
 U 1 1 5CA67677
-P 6500 4600
-F 0 "J5" H 6580 4642 50  0000 L CNN
-F 1 "PAD_Fire1" H 6580 4551 50  0000 L CNN
-F 2 "VoltMax PWM:PAD_22G" H 6500 4600 50  0001 C CNN
-F 3 "~" H 6500 4600 50  0001 C CNN
-	1    6500 4600
-	0    -1   -1   0
+P 3900 5200
+F 0 "J5" H 3980 5242 50  0000 L CNN
+F 1 "PAD_Fire1" H 3980 5151 50  0000 L CNN
+F 2 "VoltMax PWM:PAD_22G" H 3900 5200 50  0001 C CNN
+F 3 "~" H 3900 5200 50  0001 C CNN
+	1    3900 5200
+	0    1    1    0
 $EndComp
 $Comp
 L Connector_Generic:Conn_01x01 J4
 U 1 1 5CA66391
-P 5300 4600
-F 0 "J4" H 5380 4642 50  0000 L CNN
-F 1 "PAD_Fire2" H 5380 4551 50  0000 L CNN
-F 2 "VoltMax PWM:PAD_22G" H 5300 4600 50  0001 C CNN
-F 3 "~" H 5300 4600 50  0001 C CNN
-	1    5300 4600
-	0    -1   -1   0
+P 2500 5200
+F 0 "J4" H 2580 5242 50  0000 L CNN
+F 1 "PAD_Fire2" H 2580 5151 50  0000 L CNN
+F 2 "VoltMax PWM:PAD_22G" H 2500 5200 50  0001 C CNN
+F 3 "~" H 2500 5200 50  0001 C CNN
+	1    2500 5200
+	0    1    1    0
 $EndComp
 NoConn ~ 6300 3500
@@
 	6500 3050 6500 2950
 $Comp
-L Device:R R5
+L Device:R R4
 U 1 1 5CAAB1BD
 P 5550 3850
-F 0 "R5" V 5757 3850 50  0000 C CNN
+F 0 "R4" V 5757 3850 50  0000 C CNN
 F 1 "570" V 5666 3850 50  0000 C CNN
 F 2 "VoltMax PWM:R_0603_1608Metric" V 5480 3850 50  0001 C CNN
@@
 Text Label 4000 3900 1    50   ~ 0
 VIN+fromQ1Source
-Text Label 2700 4800 0    50   ~ 0
-U1toR2
-Text Label 3500 4800 0    50   ~ 0
-R2toVS
-Text Label 3900 4500 2    50   ~ 0
-R2toVS
+Text Label 2500 4700 0    50   ~ 0
+U1toS1
+Text Label 3900 4650 2    50   ~ 0
+S1toVS
 Text Label 5450 2700 0    50   ~ 0
 VIN+VM+
@@
 Wire Wire Line
 	4150 2850 4150 4800
-Connection ~ 4150 4800
-Wire Wire Line
-	4150 4800 4000 4800
 Text Label 3100 1100 0    50   ~ 0
 D2toSTR
@@
 	6100 3850 6650 3850
 Wire Wire Line
-	5150 3500 5150 5200
-Wire Wire Line
-	5150 5200 6650 5200
-Wire Wire Line
-	6650 5200 6650 4800
-Wire Wire Line
-	6650 4800 6500 4800
-Text Label 5400 5200 3    50   ~ 0
-S4VIN+toS1
+	5150 3500 5150 4800
 Wire Wire Line
 	5400 3850 5300 3850
@@
 Wire Wire Line
 	5300 3500 5400 3500
+$Comp
+L Device:R R2
+U 1 1 5C9B0658
+P 3300 4500
+F 0 "R2" V 3100 4500 50  0000 C CNN
+F 1 "10K" V 3200 4500 50  0000 C CNN
+F 2 "VoltMax PWM:R_0603_1608Metric" V 3230 4500 50  0001 C CNN
+F 3 "~" H 3300 4500 50  0001 C CNN
+	1    3300 4500
+	0    -1   -1   0
+$EndComp
+Wire Wire Line
+	5150 4800 4900 4800
+Wire Wire Line
+	2600 5100 2600 5000
+Connection ~ 2600 5000
+Connection ~ 3800 5000
+Wire Wire Line
+	3800 5000 3800 5100
+Wire Wire Line
+	2500 5000 2600 5000
+Wire Wire Line
+	3900 5000 3800 5000
+Wire Wire Line
+	3900 4100 3900 5000
+Wire Wire Line
+	3750 4100 3900 4100
+Connection ~ 3900 5000
+Wire Wire Line
+	2500 4300 2750 4300
+Connection ~ 2500 5000
+Wire Wire Line
+	4000 4800 4000 3050
+Connection ~ 4150 4800
+Wire Wire Line
+	4150 4800 4000 4800
+Wire Wire Line
+	5050 850  5050 3250
+Wire Wire Line
+	5050 3250 4250 3250
+Wire Wire Line
+	4250 3250 4250 5000
+Connection ~ 5050 850
+Wire Wire Line
+	5050 850  7000 850
+Wire Wire Line
+	3900 5000 4250 5000
+Wire Wire Line
+	2500 4300 2500 5000
+Wire Wire Line
+	2750 4300 2750 4500
+Connection ~ 2750 4300
+Wire Wire Line
+	2250 4200 2250 4750
+Connection ~ 2250 4200
+Wire Wire Line
+	2750 4500 3150 4500
+Wire Wire Line
+	3450 4500 3450 4750
+Wire Wire Line
+	3450 4750 2250 4750
+Wire Wire Line
+	1950 4750 1950 4950
+Wire Wire Line
+	1950 4750 2250 4750
+Connection ~ 2250 4750
+Wire Wire Line
+	4950 1450 4950 4200
+Text Label 3050 4500 2    50   ~ 0
+CStoR2
 $EndSCHEMATC

Commit message: Update schematic
Connections:
- wire segments 114 -> 118
Changed lines of the file:
@@
-EESchema Schematic File Version 5
+EESchema Schematic File Version 4
 LIBS:VoltMax PWM-cache
 EELAYER 29 0
@@
 L power:-BATT #PWR0101
 U 1 1 5C9FEAFF
-P 8300 4200
-F 0 "#PWR0101" H 8300 4050 50  0001 C CNN
-F 1 "-BATT" H 8315 4373 50  0000 C CNN
-F 2 "" H 8300 4200 50  0001 C CNN
-F 3 "" H 8300 4200 50  0001 C CNN
-	1    8300 4200
-	1    0    0    -1
+P 8600 4100
+F 0 "#PWR0101" H 8600 3950 50  0001 C CNN
+F 1 "-BATT" H 8450 4100 50  0000 C CNN
+F 2 "" H 8600 4100 50  0001 C CNN
+F 3 "" H 8600 4100 50  0001 C CNN
+	1    8600 4100
+	-1   0    0    1
 $EndComp
 $Comp
@@
 	1    0    0    -1
 $EndComp
-Wire Wire Line
-	8300 4200 8300 4500
 Text GLabel 8300 4300 0    50   Input ~ 0
 GND
@@
 L power:GND #PWR07
 U 1 1 5CAF4561
-P 7950 2250
-F 0 "#PWR07" H 7950 2000 50  0001 C CNN
-F 1 "GND" H 7955 2077 50  0000 C CNN
-F 2 "" H 7950 2250 50  0001 C CNN
-F 3 "" H 7950 2250 50  0001 C CNN
-	1    7950 2250
-	-1   0    0    1
+P 7800 2250
+F 0 "#PWR07" H 7800 2000 50  0001 C CNN
+F 1 "GND" H 7805 2077 50  0000 C CNN
+F 2 "" H 7800 2250 50  0001 C CNN
+F 3 "" H 7800 2250 50  0001 C CNN
+	1    7800 2250
+	1    0    0    -1
 $EndComp
 Text GLabel 7950 2400 2    50   Input ~ 0
@@
 L power:GND #PWR0102
 U 1 1 5CB29115
-P 6650 3400
-F 0 "#PWR0102" H 6650 3150 50  0001 C CNN
-F 1 "GND" H 6655 3227 50  0000 C CNN
-F 2 "" H 6650 3400 50  0001 C CNN
-F 3 "" H 6650 3400 50  0001 C CNN
-	1    6650 3400
-	-1   0    0    1
-$EndComp
-Text GLabel 6650 3550 2    50   Input ~ 0
+P 6800 3350
+F 0 "#PWR0102" H 6800 3100 50  0001 C CNN
+F 1 "GND" H 6805 3177 50  0000 C CNN
+F 2 "" H 6800 3350 50  0001 C CNN
+F 3 "" H 6800 3350 50  0001 C CNN
+	1    6800 3350
+	1    0    0    -1
+$EndComp
+Text GLabel 6650 3450 0    50   Input ~ 0
 GND
-Wire Wire Line
-	6650 3400 6650 3850
 Wire Wire Line
 	6100 3850 6650 3850
@@
 Text Label 3050 4500 2    50   ~ 0
 CStoR2
+Wire Wire Line
+	7800 2250 7950 2250
+Wire Wire Line
+	6800 3300 6800 3350
+Wire Wire Line
+	6650 3300 6650 3850
+Wire Wire Line
+	6650 3300 6800 3300
+Wire Wire Line
+	8600 4100 8300 4100
+Wire Wire Line
+	8300 4100 8300 4500
 $EndSCHEMATC
